File: Eagle/SND_SMD_Replacement.brd (EAGLE design)
At the start: 69.9 x 14.2 mm, 33 parts, among them IC1 LM358, IC2 4016D, IC3 NE555DRG4, IC4 74LVC1G06DBV, Q1 MMBT3906, Q2 MMBT3904

Commit message: Add files via upload
Parts:
- added -12V: PADS_1W_SMD, Connectors:SINGLE_CONN_SMD
- A1: value VDEV1 -> VDEV2
- D1: device SparkFun-DiscreteSemi:SOD-323 -> adafruit:SOD-123
- IC1: value LM358 -> TL072
- moved C2 0.60 mm to (16.8, 13.0)
- moved C3 0.60 mm to (24.5, 13.0)
- moved C1 0.50 mm to (29.4, 1.10)
- moved C12 0.50 mm to (24.3, 1.10)
- moved D1 0.40 mm to (26.0, 6.80)
- moved R1 0.22 mm to (29.5, 7.00)
- moved C5 0.22 mm to (29.5, 4.97)
- moved R2 0.22 mm to (29.5, 9.02)
- moved C11 0.20 mm to (12.1, 9.00)
Connections:
- new net -12V: -12V.P$1, IC1.4, Q1.3
- net GND: no longer IC1.4, Q1.3
Routing:
- net -12V: track 0.00 -> 8.75 mm, vias 0 -> 3
- net +5V: track 20.9 -> 22.2 mm
- net N$5: track 5.82 -> 6.86 mm
- net N$8: track 5.63 -> 6.60 mm
- net RES_SW: track 11.9 -> 12.8 mm
- net GND: track 35.1 -> 35.7 mm, vias 12 -> 10
- net !SND_IN: track 12.1 -> 12.8 mm
- added copper zone on layer 1, net -12V
Other:
- board size 69.9 x 14.2 mm -> 69.9 x 14.6 mm
- board text added: "-12V"
- board text added: "32 x 14.4mm"
- board text added: "GND Side"
- board text added: "SND Pin 1"
- board text added: "Sony SND SMD DosFox - VDEV2"
- board text added: "TL072"
- board text removed: "32 x 14mm"
- board text removed: "LM358"
- board text removed: "Sony SND SMD - DosFox - VDEV1"
