File: Eagle/SND_SMD_Replacement.sch (EAGLE design)
At the start: 33 parts, among them IC1 LM358, IC2 4016D, IC3 NE555DRG4, IC4 74LVC1G06DBV, Q1 MMBT3906, Q2 MMBT3904

Commit message: Add files via upload
Parts:
- added -12V: PADS_1W_SMD, Connectors:PADS_1W_SMD
- A1: value VDEV1 -> VDEV2
- D1: device SparkFun-DiscreteSemi:DIODE-ZENER-MMSZ5232BS -> adafruit:DIODESOD-123
- IC1: value LM358 -> TL072
Connections:
- new net -12V: -12V.P$1, IC1G3.P$V-, Q1.C
- net GND: no longer IC1G3.P$V-, Q1.C
Changed lines of the file:
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@@
 </classes>
 <parts>
-<part name="A1" library="Schematic Symbols" deviceset="PROJECT_DETAILS" device="_CUSTOM" value="VDEV1"/>
+<part name="A1" library="Schematic Symbols" deviceset="PROJECT_DETAILS" device="_CUSTOM" value="VDEV2"/>
 <part name="IC2" library="40xx" library_urn="urn:adsk.eagle:library:80" deviceset="4016" device="D" package3d_urn="urn:adsk.eagle:package:823/2" value="4016D"/>
 <part name="IC5" library="ICs" deviceset="SND" device=""/>
@@
 <part name="GND14" library="supply1" library_urn="urn:adsk.eagle:library:371" deviceset="GND" device=""/>
 <part name="P+11" library="Schematic Symbols" deviceset="VCC" device=""/>
-<part name="D1" library="SparkFun-DiscreteSemi" deviceset="DIODE-ZENER" device="-MMSZ5232BS" value="5.1V"/>
+<part name="D1" library="adafruit" deviceset="DIODE" device="SOD-123" value="5.1V"/>
 <part name="GND15" library="supply1" library_urn="urn:adsk.eagle:library:371" deviceset="GND" device=""/>
 <part name="R6" library="Resistors SMD" deviceset="47K_RESISTOR" device="" value="47K"/>
@@
 <part name="R5" library="Resistors SMD" deviceset="1K_RESISTOR" device="_0603" value="1k"/>
 <part name="R3" library="Resistors SMD" deviceset="GENERIC_RESISTOR" device="_0603" value="6K8"/>
-<part name="IC1" library="SparkFun-IC-Amplifiers" deviceset="OPAMP-DUAL" device="U" value="LM358"/>
+<part name="IC1" library="SparkFun-IC-Amplifiers" deviceset="OPAMP-DUAL" device="U" value="TL072"/>
 <part name="GND4" library="supply1" library_urn="urn:adsk.eagle:library:371" deviceset="GND" device=""/>
 <part name="GND7" library="supply1" library_urn="urn:adsk.eagle:library:371" deviceset="GND" device=""/>
@@
 <part name="R12" library="Resistors SMD" deviceset="150R_RESISTOR" device="_0603" value="150R"/>
 <part name="P+4" library="Schematic Symbols" deviceset="VCC" device=""/>
+<part name="GND8" library="supply1" library_urn="urn:adsk.eagle:library:371" deviceset="GND" device=""/>
+<part name="-12V" library="Connectors" deviceset="PADS_1W_SMD" device="" package3d_urn="urn:adsk.eagle:package:34340220/1"/>
 </parts>
 <sheets>
@@
 <instance part="D1" gate="G$1" x="152.4" y="86.36" smashed="yes" rot="R90">
 <attribute name="NAME" x="155.702" y="88.265" size="1.778" layer="95"/>
-<attribute name="VALUE" x="155.702" y="85.471" size="1.778" layer="96"/>
 </instance>
 <instance part="GND15" gate="1" x="152.4" y="71.12" smashed="yes">
@@
 <attribute name="VALUE" x="152.4" y="198.12" size="1.778" layer="95" font="vector" rot="R90"/>
 </instance>
-<instance part="GND4" gate="1" x="147.32" y="185.42" smashed="yes">
-<attribute name="VALUE" x="144.78" y="182.88" size="1.778" layer="96"/>
-</instance>
-<instance part="GND7" gate="1" x="347.98" y="68.58" smashed="yes">
-<attribute name="VALUE" x="345.44" y="66.04" size="1.778" layer="96"/>
-</instance>
+<instance part="GND4" gate="1" x="147.32" y="185.42" smashed="yes"/>
+<instance part="GND7" gate="1" x="347.98" y="71.12" smashed="yes"/>
 <instance part="R7" gate="R$1" x="236.22" y="121.92" smashed="yes">
 <attribute name="VALUE" x="236.22" y="124.46" size="1.778" layer="94"/>
@@
 </instance>
 <instance part="P+4" gate="+VIN" x="147.32" y="223.52" smashed="yes"/>
+<instance part="GND8" gate="1" x="86.36" y="172.72" smashed="yes"/>
+<instance part="-12V" gate="G$1" x="86.36" y="195.58" smashed="yes" rot="R90">
+<attribute name="NAME" x="83.82" y="200.66" size="1.778" layer="95"/>
+</instance>
 </instances>
 <busses>
@@
 <wire x1="33.02" y1="124.46" x2="33.02" y2="99.06" width="0.1524" layer="91"/>
 <pinref part="GND22" gate="1" pin="GND"/>
-</segment>
-<segment>
-<pinref part="IC1" gate="G3" pin="P$V-"/>
-<wire x1="147.32" y1="195.58" x2="147.32" y2="187.96" width="0.1524" layer="91"/>
-<pinref part="GND4" gate="1" pin="GND"/>
-</segment>
-<segment>
-<pinref part="GND7" gate="1" pin="GND"/>
-<wire x1="347.98" y1="71.12" x2="347.98" y2="86.36" width="0.1524" layer="91"/>
-<pinref part="Q1" gate="G$1" pin="C"/>
 </segment>
 </net>
@@
 </segment>
 </net>
+<net name="-12V" class="0">
+<segment>
+<pinref part="GND8" gate="1" pin="GND"/>
+<wire x1="86.36" y1="182.88" x2="86.36" y2="180.34" width="0.1524" layer="91"/>
+<label x="83.82" y="170.18" size="1.778" layer="95"/>
+<pinref part="-12V" gate="G$1" pin="P$1"/>
+<wire x1="86.36" y1="180.34" x2="86.36" y2="175.26" width="0.1524" layer="91"/>
+<wire x1="86.36" y1="182.88" x2="86.36" y2="187.96" width="0.1524" layer="91"/>
+</segment>
+<segment>
+<pinref part="GND7" gate="1" pin="GND"/>
+<wire x1="347.98" y1="73.66" x2="347.98" y2="86.36" width="0.1524" layer="91"/>
+<pinref part="Q1" gate="G$1" pin="C"/>
+<label x="345.44" y="68.58" size="1.778" layer="95"/>
+</segment>
+<segment>
+<pinref part="IC1" gate="G3" pin="P$V-"/>
+<wire x1="147.32" y1="195.58" x2="147.32" y2="187.96" width="0.1524" layer="91"/>
+<pinref part="GND4" gate="1" pin="GND"/>
+<label x="144.78" y="182.88" size="1.778" layer="95"/>
+</segment>
+</net>
